Commit message: add joint origin to urdf

File: utv_description/urdf/utv.urdf (robot description, URDF)
Before this commit: robot UTV, 5 links, 4 joints
Links:
- link base_link: geometry visual mesh filename=package://utv_description/meshes/UTV_frame.stl scale=0.001 0.001 0.001
- link blw: geometry visual mesh filename=package://utv_description/meshes/UTV_BLW.stl scale=0.001 0.001 0.001
- link brw: geometry visual mesh filename=package://utv_description/meshes/UTV_BRW.stl scale=0.001 0.001 0.001
- link flw: geometry visual mesh filename=package://utv_description/meshes/UTV_FLW.stl scale=0.001 0.001 0.001
- link frw: geometry visual mesh filename=package://utv_description/meshes/UTV_FRW.stl scale=0.001 0.001 0.001
Joints:
- joint base_to_blw: origin (none) -> xyz=1.45 -.6 0 rpy=0 0 0
- joint base_to_brw: origin (none) -> xyz=1.45 .6 0 rpy=0 0 0
- joint base_to_flw: origin (none) -> xyz=-.6 -.6 0 rpy=0 0 0
- joint base_to_frw: origin (none) -> xyz=-.6 .6 0 rpy=0 0 0

Commit message: test

File: utv_description/urdf/utv.urdf (robot description, URDF)
Before this commit: robot UTV, 5 links, 4 joints
Joints:
- joint base_to_brw: origin xyz=1.45 .6 0 rpy=0 0 0 -> xyz=1.46 .6 0 rpy=0 0 0

Commit message: updated joint origins

File: utv_description/urdf/utv.urdf (robot description, URDF)
Before this commit: robot UTV, 5 links, 4 joints
Joints:
- joint base_to_blw: origin xyz=1.45 -.6 0 rpy=0 0 0 -> xyz=1.39 -.615 .2919 rpy=0 0 0
- joint base_to_brw: origin xyz=1.46 .6 0 rpy=0 0 0 -> xyz=1.39 .615 .2919 rpy=0 0 0
- joint base_to_flw: origin xyz=-.6 -.6 0 rpy=0 0 0 -> xyz=-.6078 -.6237 .2919 rpy=0 0 0
- joint base_to_frw: origin xyz=-.6 .6 0 rpy=0 0 0 -> xyz=-.6078 .6237 .2919 rpy=0 0 0

Commit message: update joints and add collision

File: utv_description/urdf/utv.urdf (robot description, URDF)
Before this commit: robot UTV, 5 links, 4 joints
Links:
- link base_link: geometry collision box size=2.5 1.4 1; visual mesh filename=package://utv_description/meshes/UTV_frame.stl scale=0.001 0.001 0.001
Joints:
- joint base_to_blw: axis (none) -> 0 1 0; type fixed -> continuous
- joint base_to_brw: axis (none) -> 0 1 0; type fixed -> continuous
- joint base_to_flw: axis (none) -> 0 1 0; type fixed -> continuous
- joint base_to_frw: axis (none) -> 0 1 0; type fixed -> continuous

Commit message: added inertial values

File: utv_description/urdf/utv.urdf (robot description, URDF)
Before this commit: robot UTV, 5 links, 4 joints
Links:
- link base_link: mass None -> 1075; geometry collision box size=2.87 1.4 1.786; visual mesh filename=package://utv_description/meshes/UTV_frame.stl scale=0.001 0.001 0.001
- link blw: mass None -> 10
- link brw: mass None -> 10
- link flw: mass None -> 10
- link frw: mass None -> 10

Commit message: added xacro to urdf

File: utv_description/urdf/utv.urdf (robot description, URDF)
Before this commit: robot UTV, 5 links, 4 joints
Links:
- link base_link: mass 1075 -> ${mass}; geometry collision box size=${bodylen} ${bodywidth} ${bodyheight/2}; visual mesh filename=package://utv_description/meshes/UTV_frame.stl scale=0.001 0.001 0.001

Commit message: config files and updated urdf

File: utv_description/urdf/utv.urdf (robot description, URDF)
Before this commit: robot UTV, 5 links, 4 joints
Links:
- link base_link: mass ${mass} -> None
- link blw: mass 10 -> None
- link brw: mass 10 -> None
- link flw: mass 10 -> None
- link frw: mass 10 -> None
Joints:
- joint base_to_blw: origin xyz=1.39 -.615 .2919 rpy=0 0 0 -> xyz=1.39 -.615 .292 rpy=0 0 0
- joint base_to_brw: origin xyz=1.39 .615 .2919 rpy=0 0 0 -> xyz=1.39 .615 .292 rpy=0 0 0
- joint base_to_frw: origin xyz=-.6078 .6237 .2919 rpy=0 0 0 -> xyz=-.608 .624 .292 rpy=0 0 0

Commit message: diff drive yaml

File: utv_description/urdf/utv.urdf (robot description, URDF)
Before this commit: robot UTV, 5 links, 4 joints
Links:
- link base_link: geometry visual mesh filename=package://utv_description/meshes/UTV_frame.stl scale=0.001 0.001 0.001
- link blw: geometry collision cylinder length=${wheelthick} radius=${wheeldiam}; visual mesh filename=package://utv_description/meshes/UTV_BLW.stl scale=0.001 0.001 0.001
- link brw: geometry collision cylinder length=${wheelthick} radius=${wheeldiam}; visual mesh filename=package://utv_description/meshes/UTV_BRW.stl scale=0.001 0.001 0.001
- link flw: geometry collision cylinder length=${wheelthick} radius=${wheeldiam}; visual mesh filename=package://utv_description/meshes/UTV_FLW.stl scale=0.001 0.001 0.001
- link frw: geometry collision cylinder length=${wheelthick} radius=${wheeldiam}; visual mesh filename=package://utv_description/meshes/UTV_FRW.stl scale=0.001 0.001 0.001

Commit message: corrected collision model

File: utv_description/urdf/utv.urdf (robot description, URDF)
Before this commit: robot UTV, 5 links, 4 joints
Links:
- link base_link: geometry collision box size=${bodylen} ${bodywidth} ${bodyheight/4}; visual mesh filename=package://utv_description/meshes/UTV_frame.stl scale=0.001 0.001 0.001
- link blw: geometry collision cylinder length=${wheelthick} radius=${wheeldiam/2}; visual mesh filename=package://utv_description/meshes/UTV_BLW.stl scale=0.001 0.001 0.001
- link brw: geometry collision cylinder length=${wheelthick} radius=${wheeldiam/2}; visual mesh filename=package://utv_description/meshes/UTV_BRW.stl scale=0.001 0.001 0.001
- link flw: geometry collision cylinder length=${wheelthick} radius=${wheeldiam/2}; visual mesh filename=package://utv_description/meshes/UTV_FLW.stl scale=0.001 0.001 0.001
- link frw: geometry collision cylinder length=${wheelthick} radius=${wheeldiam/2}; visual mesh filename=package://utv_description/meshes/UTV_FRW.stl scale=0.001 0.001 0.001

Commit message: rotated frame for forward driving

File: utv_description/urdf/utv.urdf (robot description, URDF)
Before this commit: robot UTV, 5 links, 4 joints
Joints:
- joint base_to_blw: origin xyz=1.39 -.615 .292 rpy=0 0 0 -> xyz=1 -.615 .292 rpy=0 0 0
- joint base_to_brw: origin xyz=1.39 .615 .292 rpy=0 0 0 -> xyz=1 .615 .292 rpy=0 0 0
- joint base_to_flw: origin xyz=-.6078 -.6237 .2919 rpy=0 0 0 -> xyz=-1 -.6237 .2919 rpy=0 0 0
- joint base_to_frw: origin xyz=-.608 .624 .292 rpy=0 0 0 -> xyz=-1 .624 .292 rpy=0 0 0

Commit message: new model and updated urdf

File: utv_description/urdf/utv.urdf (robot description, URDF)
Before this commit: robot UTV, 5 links, 4 joints
Links:
- link base_link: geometry collision box size=${utvlen} ${utvwidth} ${utvheight/4}; visual mesh filename=package://utv_description/meshes/UTV_frame.stl
- link blw: geometry collision cylinder length=${wheelthick} radius=${wheeldiam/2}; visual mesh filename=package://utv_description/meshes/UTV_BLW.stl
- link brw: geometry collision cylinder length=${wheelthick} radius=${wheeldiam/2}; visual mesh filename=package://utv_description/meshes/UTV_BRW.stl
- link flw: geometry collision cylinder length=${wheelthick} radius=${wheeldiam/2}; visual mesh filename=package://utv_description/meshes/UTV_FLW.stl
- link frw: geometry collision cylinder length=${wheelthick} radius=${wheeldiam/2}; visual mesh filename=package://utv_description/meshes/UTV_FRW.stl
Joints:
- joint base_to_blw: origin xyz=1 -.615 .292 rpy=0 0 0 -> xyz=-1 -.62 .29 rpy=0 0 0
- joint base_to_brw: origin xyz=1 .615 .292 rpy=0 0 0 -> xyz=-1 .62 .29 rpy=0 0 0
- joint base_to_flw: origin xyz=-1 -.6237 .2919 rpy=0 0 0 -> xyz=1 -.62 .29 rpy=0 0 0
- joint base_to_frw: origin xyz=-1 .624 .292 rpy=0 0 0 -> xyz=1 .62 .29 rpy=0 0 0

Commit message: clean up urdf

File: utv_description/urdf/utv.urdf (robot description, URDF)
Before this commit: robot UTV, 5 links, 4 joints
Links:
- removed link flw
- removed link frw
Joints:
- joint base_to_flw: origin xyz=1 -.62 .29 rpy=0 0 0 -> xyz=1 .62 .29 rpy=0 0 0
- joint base_to_frw: origin xyz=1 .62 .29 rpy=0 0 0 -> xyz=1 -.62 .29 rpy=0 0 0
