Commit message: update urdf and ackermann steering

File: utv_description/urdf/utv_steer.urdf (robot description, URDF)
Before this commit: robot UTV, 5 links, 4 joints
Links:
- added link front_steer
- added link rear_steer
- added link steer_left
- added link steer_right
Joints:
- added joint front_steer_joint: type fixed, parent base_link, child front_steer, origin xyz=1 0 .29  rpy=0 0 0, axis 0 0 1
- added joint rear_steer_joint: type continuous, parent base_link, child rear_steer, origin xyz=-1 0 .29  rpy=0 0 0, axis 0 1 0
- added joint steer_left_joint: type revolute, parent base_link, child steer_left, origin xyz=1 .62 .5  rpy=0 0 0, axis 0 0 1, limit lower=-${pi/2} upper=${pi/2} effort=10 velocity=1
- added joint steer_right_joint: type revolute, parent base_link, child steer_right, origin xyz=1 -.62 .5  rpy=0 0 0, axis 0 0 1, limit lower=-${pi/2} upper=${pi/2} effort=10 velocity=1
