Commit message: added required dependencies

File: vehicle_model/urdf/body.xacro (robot description, xacro)
@@ -31,7 +31,7 @@
       </visual>
       <collision>
-        <origin xyz="${wheel_base/2} 0 ${vehicle_height/2}" rpy="0 0 0"/>
+        <origin xyz="0 0 ${vehicle_height/3}" rpy="0 0 0"/>
         <geometry>
-          <box size="${vehicle_length} 0.9 ${vehicle_height}"/>
+          <box size="${vehicle_length} 0.9 ${vehicle_height/2}"/>
         </geometry>
       </collision>

File: vehicle_model/urdf/wheel.xacro (robot description, xacro)
@@ -29,5 +29,5 @@
       </inertial>
       <collision>
-        <origin xyz="0 0 0" rpy="0 ${pi/2} 0"/>
+        <origin xyz="0 0 0" rpy="${pi/2} 0 0"/>
         <geometry>
           <cylinder radius="${radius}" length="${width}" />
